Commit message: add leuze

File: src/hao_urdf/urdf/hao_body.xacro (robot description, xacro)
@@ -1,4 +1,4 @@
 <?xml version="1.0"?>
-<robot name="mbot" xmlns:xacro="http://www.ros.org/wiki/xacro">
+<robot name="hao" xmlns:xacro="http://www.ros.org/wiki/xacro">
   <!-- PROPERTY LIST -->
   <xacro:property name="M_PI" value="3.14159" />
@@ -7,11 +7,11 @@
   <xacro:property name="motor_length" value="0.08" />
   <xacro:property name="motor_x" value="0" />
-  <xacro:property name="motor_y" value="0.075" />
+  <xacro:property name="motor_y" value="0.185" />
   <xacro:property name="wheel_mass" value="2" />
-  <xacro:property name="wheel_radius" value="0.033" />
+  <xacro:property name="wheel_radius" value="0.08" />
   <xacro:property name="wheel_length" value="0.017" />
   <xacro:property name="wheel_y" value="${(motor_length+wheel_length)/2}" />
   <xacro:property name="plate_mass" value="2" />
-  <xacro:property name="plate_radius" value="0.13" />
+  <xacro:property name="plate_radius" value="0.3" />
   <xacro:property name="plate_length" value="0.005" />
   <xacro:property name="plate_height" value="0.07" />
@@ -70,5 +70,5 @@
               <origin xyz="0 0 0" rpy="0 0 0" />
               <geometry>
-                  <cylinder radius="${plate_radius}" length="${plate_length}" />
+                  <box size="0.58 0.44 0.005"/>
               </geometry>
               <material name="yellow" />
@@ -77,5 +77,5 @@
               <origin xyz="0 0 0" rpy="0 0 0" />
               <geometry>
-                  <cylinder radius="${plate_radius}" length="${plate_length}" />
+                  <box size="0.58 0.44 0.03"/>
               </geometry>
           </collision>
@@ -203,5 +203,5 @@
             <origin xyz="0 0 0" rpy="0 0 0" />
             <geometry>
-                <cylinder radius="${plate_radius}" length="${plate_length}" />
+                <box size="0.58 0.44 0.005"/>
             </geometry>
             <material name="yellow" />
@@ -210,5 +210,5 @@
             <origin xyz="0 0 0" rpy="0 0 0" />
             <geometry>
-                <cylinder radius="${plate_radius}" length = "${plate_length}"/>
+               <box size="0.58 0.44 0.005"/>
             </geometry>
         </collision>

File: src/hao_urdf/urdf/hao_slamopto.xacro (robot description, xacro)
@@ -7,6 +7,6 @@
 	<xacro:property name="kinect_offset_y" value="0" />
 	<xacro:property name="kinect_offset_z" value="0.035" />
-  <xacro:property name="rplidar_offset_x1" value="-0.15" />
-  <xacro:property name="rplidar_offset_x2" value="0.15" />
+  <xacro:property name="rplidar_offset_x1" value="-0.20" />
+  <xacro:property name="rplidar_offset_x2" value="0.20" />
 	<xacro:property name="rplidar_offset_y" value="0" />
 	<xacro:property name="rplidar_offset_z" value="0.028" />
