Commit message: update hw to hw5

File: src/homework/hw5/urdf/myRobot.urdf (robot description, URDF)
Before this commit: robot myRobot, 14 links, 13 joints
Links:
- link RGBD_camera_link: geometry visual mesh filename=package://hw5/meshes/kinect.dae
- link gps_link: geometry visual mesh filename=package://hw5/meshes/dae/gps_link.dae
- link left_camera_bracket_link: geometry visual mesh filename=package://hw5/meshes/dae/left_camera_slide.dae
- link left_camera_link: geometry visual mesh filename=package://hw5/meshes/dae/camera.dae
- link lidar_bracket_link: geometry visual mesh filename=package://hw5/meshes/dae/lidar_bracket_link.dae
- link right_camera_bracket_link: geometry visual mesh filename=package://hw5/meshes/dae/right_camera_slide.dae
- link right_camera_link: geometry visual mesh filename=package://hw5/meshes/dae/camera.dae
